File: Z Axis Motor Driver.sch (KiCad schematic (older format))
At the start: 6 parts

Commit message: Finished TMC2209 schematic for Y and Z motor, added BOM
Parts:
- added C? (x2): 100nF, Capacitor_SMD:C_0603_1608Metric, symbol Device:C_Small
- added C? (x4): 470p, Capacitor_SMD:C_0603_1608Metric, symbol Device:C_Small
- added C?: 330u, symbol Device:CP_Small
- added C?: 10u, symbol Device:C_Small
- added C?: 100n, Capacitor_SMD:C_0603_1608Metric, symbol Device:C_Small
- added C?: 1u, symbol Device:C_Small
- added C?: 2.2u, Capacitor_SMD:C_0603_1608Metric, symbol Device:C_Small
- added D? (x8): SK25, Diode_SMD:D_SMB, symbol Device:D_Schottky_ALT
- added FB? (x4): 60Ohm@100MHz, Inductor_SMD:L_0805_2012Metric, symbol Device:Ferrite_Bead_Small
- added J?: Motor Z, Connector_JST:JST_XH_B4B-XH-AM_1x04_P2.50mm_Vertical, symbol Connector:Conn_01x04_Male
- added R?: 1k, Resistor_SMD:R_0603_1608Metric, symbol Device:R
- added R?: 100k, Resistor_SMD:R_0603_1608Metric, symbol Device:R
- added TP?: Z_OB2, symbol Connector:TestPoint
- added TP?: Z_OB1, symbol Connector:TestPoint
- added TP?: Z_OA2, symbol Connector:TestPoint
- added TP?: Z_OA1, symbol Connector:TestPoint
- C?: footprint Capacitor_SMD:C_0805_2012Metric -> Capacitor_SMD:C_0603_1608Metric; Tolerancja 10% -> (none)
Connections:
- net labels added: UART_RX, UART_TX, VS, Z_DIAG, Z_DIR, Z_ENN, Z_INDEX, Z_STEP
- net labels removed: VSS
- wire segments 30 -> 125
- no-connect marks 0 -> 6
Other:
- note added: "EMC"
- note added: "ESD"
- note added: "INDEX na wejście Timera STM"
- note added: "Low ESR electrolytic capacitors\nare recommended for VS filtering."
- note added: "Motor Z output"
- note added: "Pin 25 NC można podłączyć do GND jeśli poprawi to rutowanie PCB"
- note added: "Place near IC with\nshort path to die pad"
- note added: "Wybrać address"
- note added: "Zabezpieczenie EMC może zredukować zakłócenia elektromagnetyczne, przetestować czy warto jest stosować."
- note added: "Zabezpieczenie ESD można pominąć gdy silnik nie będzie wpinany/rozpinany hot-plug"
- note added: "Złącze JST XH2.5"
- note removed: "ESD Protection"
- moved on the sheet: C?, R?, U?
