File: Z Axis Motor Driver.sch (KiCad schematic (older format))
At the start: 34 parts, among them J2 Motor Z, U2 TMC2209-LA

Commit message: Start TMC routing
Parts:
- removed TP5: Z_OB2, TestPoint:TestPoint_Pad_D1.5mm, symbol Connector:TestPoint
- removed TP6: Z_OB1, TestPoint:TestPoint_Pad_D1.5mm, symbol Connector:TestPoint
- removed TP7: Z_OA2, TestPoint:TestPoint_Pad_D1.5mm, symbol Connector:TestPoint
- removed TP8: Z_OA1, TestPoint:TestPoint_Pad_D1.5mm, symbol Connector:TestPoint
Connections:
- net at U2.1 (OB2): now also FB5.2; no longer FB8.2
- net at U2.21 (OA2): now also FB8.2; no longer FB6.2
- net at U2.24 (OA1): now also FB7.2; no longer FB5.2
- net at U2.26 (OB1): now also FB6.2; no longer FB7.2
Changed lines of the file:
@@
 	0    1    1    0
 $EndComp
-Wire Wire Line
-	4400 3550 6050 3550
-Wire Wire Line
-	6050 3550 6050 3050
-Wire Wire Line
-	4400 3450 5950 3450
-Wire Wire Line
-	5950 3450 5950 2900
 $Comp
 L Device:C_Small C28
@@
 	1    0    0    -1
 $EndComp
-Wire Wire Line
-	9200 2900 9200 3300
-Wire Wire Line
-	8850 3050 8850 3300
 Connection ~ 8500 3600
 Connection ~ 8850 3050
@@
 Text Notes 10150 2850 0    50   ~ 0
 Złącze JST XH2.5
-Wire Wire Line
-	8150 3750 8150 3300
-$Comp
-L Connector:TestPoint TP5
-U 1 1 5E0831DE
-P 8150 3300
-F 0 "TP5" V 8050 3350 50  0000 L CNN
-F 1 "Z_OB2" V 8250 3350 50  0000 L CNN
-F 2 "TestPoint:TestPoint_Pad_D1.5mm" H 8350 3300 50  0001 C CNN
-F 3 "~" H 8350 3300 50  0001 C CNN
-	1    8150 3300
-	0    1    1    0
-$EndComp
-$Comp
-L Connector:TestPoint TP6
-U 1 1 5E087114
-P 8500 3300
-F 0 "TP6" V 8400 3350 50  0000 L CNN
-F 1 "Z_OB1" V 8600 3350 50  0000 L CNN
-F 2 "TestPoint:TestPoint_Pad_D1.5mm" H 8700 3300 50  0001 C CNN
-F 3 "~" H 8700 3300 50  0001 C CNN
-	1    8500 3300
-	0    1    1    0
-$EndComp
-Wire Wire Line
-	8500 3300 8500 3600
-$Comp
-L Connector:TestPoint TP7
-U 1 1 5E0874C7
-P 8850 3300
-F 0 "TP7" V 8750 3350 50  0000 L CNN
-F 1 "Z_OA2" V 8950 3350 50  0000 L CNN
-F 2 "TestPoint:TestPoint_Pad_D1.5mm" H 9050 3300 50  0001 C CNN
-F 3 "~" H 9050 3300 50  0001 C CNN
-	1    8850 3300
-	0    1    1    0
-$EndComp
-$Comp
-L Connector:TestPoint TP8
-U 1 1 5E087849
-P 9200 3300
-F 0 "TP8" V 9100 3350 50  0000 L CNN
-F 1 "Z_OA1" V 9300 3350 50  0000 L CNN
-F 2 "TestPoint:TestPoint_Pad_D1.5mm" H 9400 3300 50  0001 C CNN
-F 3 "~" H 9400 3300 50  0001 C CNN
-	1    9200 3300
-	0    1    1    0
-$EndComp
 Text GLabel 1400 2850 0    50   Input ~ 0
 Z_STEP
@@
 	2700 2950 1400 2950
 Wire Wire Line
-	6150 3650 6150 3600
-Wire Wire Line
-	4400 3650 6150 3650
-Wire Wire Line
 	7050 2900 7300 2900
 Wire Wire Line
@@
 	7700 3050 8850 3050
 Wire Wire Line
-	6150 3600 6850 3600
-Wire Wire Line
-	4400 3750 6850 3750
+	6250 3600 6850 3600
 Wire Wire Line
 	6050 3050 6850 3050
@@
 	0    1    1    0
 $EndComp
-Wire Wire Line
-	9200 3300 9200 4100
 $Comp
 L Device:D_TVS_ALT D?
@@
 	8050 4050 9500 4050
 Wire Wire Line
-	8850 3300 8850 4100
-Wire Wire Line
 	9200 4400 9200 5000
 $Comp
@@
 Wire Wire Line
 	8500 3600 8500 4100
-Connection ~ 8850 3300
-Connection ~ 9200 3300
 $Comp
 L Device:D_TVS_ALT D?
@@
 Wire Wire Line
 	9750 3750 9750 4100
+Wire Wire Line
+	4400 3750 5950 3750
+Wire Wire Line
+	5950 2900 5950 3750
+Wire Wire Line
+	6050 3650 4400 3650
+Wire Wire Line
+	6050 3050 6050 3650
+Wire Wire Line
+	4400 3450 6250 3450
+Wire Wire Line
+	6250 3450 6250 3600
+Wire Wire Line
+	6850 3750 6150 3750
+Wire Wire Line
+	6150 3750 6150 3550
+Wire Wire Line
+	6150 3550 4400 3550
+Wire Wire Line
+	8850 3050 8850 4100
+Wire Wire Line
+	9200 2900 9200 4100
 $EndSCHEMATC

Commit message: TMC2209 routing step 2/3
Parts:
- removed C15: 330uF, Capacitor_THT:CP_Radial_D10.0mm_P5.00mm, symbol Device:CP_Small
- added C90, C91: 120uF, Capacitor_THT:CP_Radial_D8.0mm_P3.50mm, symbol Device:CP_Small
- added C92: 10uF, Capacitor_SMD:C_1210_3225Metric, symbol Device:C_Small
Connections:
- net GND: now also C90.2, C91.2, C92.2; no longer R7.1
- net VCC: now also R7.1
- net VS: now also C90.1, C91.1, C92.1
Other:
- moved on the sheet: C16, C17, C18

Commit message: Added 3d packages, improved TMC2209 footprint
Parts:
- U2: footprint footprints:QFN-28_5X5_3X8_EPAD -> footprints:QFN-28_5X5mm_P0.5mm_EP3.35x.3.35mm
Changed lines of the file:
@@
 F 0 "U2" H 2650 4700 60  0000 L CNN
 F 1 "TMC2209-LA" H 2650 4600 60  0000 L CNN
-F 2 "footprints:QFN-28_5X5_3X8_EPAD" V 3500 3600 60  0001 C CNN
+F 2 "footprints:QFN-28_5X5mm_P0.5mm_EP3.35x.3.35mm" V 3500 3600 60  0001 C CNN
 F 3 "https://www.trinamic.com/fileadmin/assets/Products/ICs_Documents/TMC2209_Datasheet_V103.pdf" H 2500 4250 60  0001 C CNN
 F 4 "10.30" H 3550 3600 50  0001 C CNN "Cena"

Commit message: Updated BOM on schematics
Parts:
- C16, C92: Link (none) -> https://www.tme.eu/pl/details/cl32b106kbjnnne/kondensatory-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; Opis (none) -> Kondensator: ceramiczny; MLCC; 10uF; 50V; X7R; ±10%; SMD; 1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
- C17: Link (none) -> https://www.tme.eu/pl/details/cl21b105kbfnnng/kondensatory-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; Opis (none) -> Kondensator: ceramiczny; MLCC; 1uF; 50V; X7R; ±10%; SMD; 08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
- C18, C19, C20, C22, C24: Cena 0.05982 -> 0.07894; Link (none) -> https://www.tme.eu/pl/details/cl10b104kb8nnnc/kondensatory-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; Model CL10B104KB8NNNC -> CL10B104KB8NNNC; Opis (none) -> Kondensator: ceramiczny; MLCC; 100nF; 50V; X7R; ±10%; SMD; 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
- C21: Opis (none) -> Kondensator: ceramiczny; MLCC; 22nF; 50V; X7R; ±10%; SMD; 0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
- C23: Opis (none) -> Kondensator: ceramiczny; MLCC; 2,2uF; 10V; X5R; ±10%; SMD; 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
- C25, C26, C27, C28: Opis (none) -> Kondensator: ceramiczny; MLCC; 470pF; 100VDC; C0G; ±5%; SMD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
- R7: Link (none) -> https://www.tme.eu/pl/details/smd0603-100k-1%25/rezystory-s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; Model (none) -> 0603SAF1003T5E; Opis (none) -> Rezystor: thick film; SMD; 0603; 100kΩ; 0,1W; ±1%; -55÷155°C; Producent (none) -> ROYAL OHM
Changed lines of the file:
@@
 F 10 "10%" H 4850 3050 50  0001 C CNN "Tolerancja"
 F 11 "SMD" H 4850 3050 50  0001 C CNN "Typ"
+F 12 "Kondensator: ceramiczny; MLCC; 22nF; 50V; X7R; ±10%; SMD; 0603" H 4850 3050 50  0001 C CNN "Opis"
 	1    4850 3050
 	1    0    0    -1
@@
 F 5 "X7R" H 3450 2000 50  0000 L CNN "Dielektryk"
 F 6 "10%" H 3450 1900 50  0000 L CNN "Tolerancja"
-F 7 "CL10B104KB8NNNC " H 3350 2050 50  0001 C CNN "Model"
-F 8 "0.05982" H 3350 2050 50  0001 C CNN "Cena"
+F 7 "CL10B104KB8NNNC" H 3350 2050 50  0001 C CNN "Model"
+F 8 "0.07894" H 3350 2050 50  0001 C CNN "Cena"
 F 9 "SAMSUNG" H 3350 2050 50  0001 C CNN "Producent"
 F 10 "SMD" H 3350 2050 50  0001 C CNN "Typ"
+F 11 "https://www.tme.eu/pl/details/cl10b104kb8nnnc/kondensatory-mlcc-smd-0603/samsung/" H 3350 2050 50  0001 C CNN "Link"
+F 12 "Kondensator: ceramiczny; MLCC; 100nF; 50V; X7R; ±10%; SMD; 0603" H 3350 2050 50  0001 C CNN "Opis"
 	1    3350 2050
 	1    0    0    -1
@@
 F 5 "X7R" H 4050 2000 50  0000 L CNN "Dielektryk"
 F 6 "10%" H 4050 1900 50  0000 L CNN "Tolerancja"
-F 7 "CL10B104KB8NNNC " H 3950 2050 50  0001 C CNN "Model"
-F 8 "0.05982" H 3950 2050 50  0001 C CNN "Cena"
+F 7 "CL10B104KB8NNNC" H 3950 2050 50  0001 C CNN "Model"
+F 8 "0.07894" H 3950 2050 50  0001 C CNN "Cena"
 F 9 "SAMSUNG" H 3950 2050 50  0001 C CNN "Producent"
 F 10 "SMD" H 3950 2050 50  0001 C CNN "Typ"
+F 11 "https://www.tme.eu/pl/details/cl10b104kb8nnnc/kondensatory-mlcc-smd-0603/samsung/" H 3950 2050 50  0001 C CNN "Link"
+F 12 "Kondensator: ceramiczny; MLCC; 100nF; 50V; X7R; ±10%; SMD; 0603" H 3950 2050 50  0001 C CNN "Opis"
 	1    3950 2050
 	1    0    0    -1
@@
 F 5 "X7R" H 5292 4209 50  0000 L CNN "Dielektryk"
 F 6 "10%" H 5292 4118 50  0000 L CNN "Tolerancja"
-F 7 "CL10B104KB8NNNC " H 5200 4300 50  0001 C CNN "Model"
-F 8 "0.05982" H 5200 4300 50  0001 C CNN "Cena"
+F 7 "CL10B104KB8NNNC" H 5200 4300 50  0001 C CNN "Model"
+F 8 "0.07894" H 5200 4300 50  0001 C CNN "Cena"
 F 9 "SAMSUNG" H 5200 4300 50  0001 C CNN "Producent"
 F 10 "SMD" H 5200 4300 50  0001 C CNN "Typ"
+F 11 "https://www.tme.eu/pl/details/cl10b104kb8nnnc/kondensatory-mlcc-smd-0603/samsung/" H 5200 4300 50  0001 C CNN "Link"
+F 12 "Kondensator: ceramiczny; MLCC; 100nF; 50V; X7R; ±10%; SMD; 0603" H 5200 4300 50  0001 C CNN "Opis"
 	1    5200 4300
 	1    0    0    -1
@@
 F 5 "X7R" H 6342 4209 50  0000 L CNN "Dielektryk"
 F 6 "10%" H 6342 4118 50  0000 L CNN "Tolerancja"
-F 7 "CL10B104KB8NNNC " H 6250 4300 50  0001 C CNN "Model"
-F 8 "0.05982" H 6250 4300 50  0001 C CNN "Cena"
+F 7 "CL10B104KB8NNNC" H 6250 4300 50  0001 C CNN "Model"
+F 8 "0.07894" H 6250 4300 50  0001 C CNN "Cena"
 F 9 "SAMSUNG" H 6250 4300 50  0001 C CNN "Producent"
 F 10 "SMD" H 6250 4300 50  0001 C CNN "Typ"
+F 11 "https://www.tme.eu/pl/details/cl10b104kb8nnnc/kondensatory-mlcc-smd-0603/samsung/" H 6250 4300 50  0001 C CNN "Link"
+F 12 "Kondensator: ceramiczny; MLCC; 100nF; 50V; X7R; ±10%; SMD; 0603" H 6250 4300 50  0001 C CNN "Opis"
 	1    6250 4300
 	1    0    0    -1
@@
 F 10 "KEMET" H 7700 4250 50  0001 C CNN "Producent"
 F 11 "SMD" H 7700 4250 50  0001 C CNN "Typ"
+F 12 "Kondensator: ceramiczny; MLCC; 470pF; 100VDC; C0G; ±5%; SMD; 0805" H 7700 4250 50  0001 C CNN "Opis"
 	1    7700 4250
 	1    0    0    -1
@@
 F 10 "KEMET" H 7300 2500 50  0001 C CNN "Producent"
 F 11 "SMD" H 7300 2500 50  0001 C CNN "Typ"
+F 12 "Kondensator: ceramiczny; MLCC; 470pF; 100VDC; C0G; ±5%; SMD; 0805" H 7300 2500 50  0001 C CNN "Opis"
 	1    7300 2500
 	1    0    0    -1
@@
 F 10 "KEMET" H 7300 4250 50  0001 C CNN "Producent"
 F 11 "SMD" H 7300 4250 50  0001 C CNN "Typ"
+F 12 "Kondensator: ceramiczny; MLCC; 470pF; 100VDC; C0G; ±5%; SMD; 0805" H 7300 4250 50  0001 C CNN "Opis"
 	1    7300 4250
 	1    0    0    -1
@@
 F 10 "KEMET" H 7700 2500 50  0001 C CNN "Producent"
 F 11 "SMD" H 7700 2500 50  0001 C CNN "Typ"
+F 12 "Kondensator: ceramiczny; MLCC; 470pF; 100VDC; C0G; ±5%; SMD; 0805" H 7700 2500 50  0001 C CNN "Opis"
 	1    7700 2500
 	1    0    0    -1
@@
 F 9 "10%" H 1800 2050 50  0001 C CNN "Tolerancja"
 F 10 "SMD" H 1800 2050 50  0001 C CNN "Typ"
+F 11 "https://www.tme.eu/pl/details/cl32b106kbjnnne/kondensatory-mlcc-smd-1210/samsung/" H 1800 2050 50  0001 C CNN "Link"
+F 12 "Kondensator: ceramiczny; MLCC; 10uF; 50V; X7R; ±10%; SMD; 1210" H 1800 2050 50  0001 C CNN "Opis"
 	1    1800 2050
 	1    0    0    -1
@@
 F 4 "50V" H 2950 2000 50  0000 L CNN "Napięcie"
 F 5 "X7R" H 2950 1900 50  0000 L CNN "Dielektryk"
-F 6 "0.05982" H 2850 2050 50  0001 C CNN "Cena"
-F 7 "CL10B104KB8NNNC " H 2850 2050 50  0001 C CNN "Model"
+F 6 "0.07894" H 2850 2050 50  0001 C CNN "Cena"
+F 7 "CL10B104KB8NNNC" H 2850 2050 50  0001 C CNN "Model"
 F 8 "SAMSUNG" H 2850 2050 50  0001 C CNN "Producent"
 F 9 "10%" H 2850 2050 50  0001 C CNN "Tolerancja"
 F 10 "SMD" H 2850 2050 50  0001 C CNN "Typ"
+F 11 "https://www.tme.eu/pl/details/cl10b104kb8nnnc/kondensatory-mlcc-smd-0603/samsung/" H 2850 2050 50  0001 C CNN "Link"
+F 12 "Kondensator: ceramiczny; MLCC; 100nF; 50V; X7R; ±10%; SMD; 0603" H 2850 2050 50  0001 C CNN "Opis"
 	1    2850 2050
 	1    0    0    -1
@@
 F 9 "10%" H 2500 2050 50  0001 C CNN "Tolerancja"
 F 10 "SMD" H 2500 2050 50  0001 C CNN "Typ"
+F 11 "https://www.tme.eu/pl/details/cl21b105kbfnnng/kondensatory-mlcc-smd-0805/samsung/" H 2500 2050 50  0001 C CNN "Link"
+F 12 "Kondensator: ceramiczny; MLCC; 1uF; 50V; X7R; ±10%; SMD; 0805" H 2500 2050 50  0001 C CNN "Opis"
 	1    2500 2050
 	1    0    0    -1
@@
 F 9 "SAMSUNG" H 5250 3050 50  0001 C CNN "Producent"
 F 10 "SMD" H 5250 3050 50  0001 C CNN "Typ"
+F 11 "Kondensator: ceramiczny; MLCC; 2,2uF; 10V; X5R; ±10%; SMD; 0603" H 5250 3050 50  0001 C CNN "Opis"
 	1    5250 3050
 	1    0    0    -1
@@
 F 2 "Resistor_SMD:R_0603_1608Metric" V 2130 4550 50  0001 C CNN
 F 3 "~" H 2200 4550 50  0001 C CNN
-F 4 "" H 2200 4550 50  0001 C CNN "Model"
+F 4 "0603SAF1003T5E" H 2200 4550 50  0001 C CNN "Model"
 F 5 "0.04651" H 2200 4550 50  0001 C CNN "Cena"
 F 6 "SMD" H 2200 4550 50  0001 C CNN "Typ"
+F 7 "https://www.tme.eu/pl/details/smd0603-100k-1%25/rezystory-smd-0603/royal-ohm/0603saf1003t5e/" H 2200 4550 50  0001 C CNN "Link"
+F 8 "Rezystor: thick film; SMD; 0603; 100kΩ; 0,1W; ±1%; -55÷155°C" H 2200 4550 50  0001 C CNN "Opis"
+F 9 "ROYAL OHM" H 2200 4550 50  0001 C CNN "Producent"
 	1    2200 4550
 	-1   0    0    1
@@
 F 9 "10%" H 2150 2050 50  0001 C CNN "Tolerancja"
 F 10 "SMD" H 2150 2050 50  0001 C CNN "Typ"
+F 11 "https://www.tme.eu/pl/details/cl32b106kbjnnne/kondensatory-mlcc-smd-1210/samsung/" H 2150 2050 50  0001 C CNN "Link"
+F 12 "Kondensator: ceramiczny; MLCC; 10uF; 50V; X7R; ±10%; SMD; 1210" H 2150 2050 50  0001 C CNN "Opis"
 	1    2150 2050
 	1    0    0    -1
