File: Microcontroller.sch (KiCad schematic (older format))
At the start: 32 parts, among them J3 USB_B, J4 SWD, J5 DEBUG, Q1 BC817, U3 USBUF02W6, U4 STM32F401VETx, Y1 8MHz

Commit message: Shematic almost finished, BOM in KiCad 3/4 finished
Parts:
- C29: renamed from C35; footprint (none) -> Capacitor_SMD:C_0603_1608Metric; Cena (none) -> 0.14766; Link (none) -> https://www.tme.eu/pl/details/c0603c200j5gac/kondensatory-m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; Model (none) -> C0603C200J5GAC; Napięcie (none) -> 16V; Producent (none) -> KEMET; Typ (none) -> SMD
- C30: renamed from C36; footprint (none) -> Capacitor_SMD:C_0603_1608Metric; Cena (none) -> 0.14766; Link (none) -> https://www.tme.eu/pl/details/c0603c200j5gac/kondensatory-m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; Model (none) -> C0603C200J5GAC; Napięcie (none) -> 16V; Producent (none) -> KEMET; Typ (none) -> SMD
- C31: renamed from C32; footprint (none) -> Capacitor_SMD:C_0603_1608Metric; Cena (none) -> 0.05982; Model (none) -> CL10B104KB8NNNC; Napięcie (none) -> 50V; Producent (none) -> SAMSUNG; Tolerancja (none) -> 10%; Typ (none) -> SMD
- C32: renamed from C33; footprint (none) -> Capacitor_SMD:C_0603_1608Metric; Cena (none) -> 0.08; Link (none) -> https://www.tme.eu/pl/details/cl10a225kp8nnnc/kondensatory-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; Model (none) -> CL10A225KP8NNNC; Napięcie (none) -> 6.3V; Producent (none) -> SAMSUNG; Typ (none) -> SMD
- C33: renamed from C34; footprint (none) -> Capacitor_SMD:C_0603_1608Metric; Cena (none) -> 0.08; Link (none) -> https://www.tme.eu/pl/details/cl10a225kp8nnnc/kondensatory-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; Model (none) -> CL10A225KP8NNNC; Napięcie (none) -> 6.3V; Producent (none) -> SAMSUNG; Typ (none) -> SMD
- C34: renamed from C31; footprint (none) -> Capacitor_SMD:C_0603_1608Metric; Cena (none) -> 0.05982; Model (none) -> CL10B104KB8NNNC; Napięcie (none) -> 50V; Producent (none) -> SAMSUNG; Tolerancja (none) -> 10%; Typ (none) -> SMD
- C35: renamed from C29; footprint (none) -> Capacitor_SMD:C_0603_1608Metric; Cena (none) -> 0.05982; Model (none) -> CL10B104KB8NNNC; Napięcie (none) -> 50V; Producent (none) -> SAMSUNG; Tolerancja (none) -> 10%; Typ (none) -> SMD
- C36: renamed from C30; footprint (none) -> Capacitor_SMD:C_0603_1608Metric; Cena (none) -> 0.09; Dielektryk (none) -> X7R; Model (none) -> CL21B105KBFNNNE; Napięcie (none) -> 50V; Producent (none) -> SAMSUNG; Tolerancja (none) -> 10%; Typ (none) -> SMD
- C37, C38, C39, C40, C41, C42: footprint (none) -> Capacitor_SMD:C_0603_1608Metric; Cena (none) -> 0.05982; Model (none) -> CL10B104KB8NNNC; Napięcie (none) -> 50V; Producent (none) -> SAMSUNG; Tolerancja (none) -> 10%; Typ (none) -> SMD
- D17: Cena (none) -> 0.34; Link (none) -> https://www.tme.eu/pl/details/of-smd2012g-1/diody-led-smd-k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; Model (none) -> OF-SMD2012G-1; Opis (none) -> LED; SMD; 0805; zielony; 600÷800mcd; 2x1,25x0,68mm; 120°; 2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; Producent (none) -> OPTOFLASH; Typ (none) -> SMD
- J5: footprint Connector_JST:JST_PH_B2B-PH-K_1x03_P2.00mm_Vertical -> Connector_JST:JST_PH_B3B-PH-K_1x03_P2.00mm_Vertical; Cena (none) -> 0.59599; Link (none) -> https://www.tme.eu/pl/details/b3b-ph-k-s/zlacza-sygnalowe-r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; Model (none) -> B3B-PH-K-S; Opis (none) -> Gniazdo; przewód-płytka; męskie; PH; 2mm; PIN: 3; THT; 100V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; Producent (none) -> JST; Typ (none) -> THT
- R10: renamed from R15; footprint (none) -> Resistor_SMD:R_0603_1608Metric
- R11: renamed from R14; footprint (none) -> Resistor_SMD:R_0603_1608Metric
- R12: footprint (none) -> Resistor_SMD:R_0603_1608Metric
- R13: renamed from R10; footprint (none) -> Resistor_SMD:R_0603_1608Metric
- R14: renamed from R11; footprint (none) -> Resistor_SMD:R_0603_1608Metric
- R15: renamed from R17; footprint (none) -> Resistor_SMD:R_0603_1608Metric
- R16: renamed from R13; footprint (none) -> Resistor_SMD:R_0603_1608Metric
- R17: renamed from R16; footprint (none) -> Resistor_SMD:R_0603_1608Metric
- U3: renamed from U4; Cena (none) -> 22.53; Link (none) -> https://pl.farnell.com/stmicroelectronics/stm32f401vbt6/mcu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; Model (none) -> STM32F401VBT6; Opis (none) -> ARM MCU, linia Dynamic Efficiency, STM32 Family STM32F4 Ser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; Producent (none) -> STM; Typ (none) -> SMD
- U4: renamed from U3; Cena (none) -> 1.0587; Link (none) -> https://www.tme.eu/pl/details/usbuf02w6/filtry-uklady-scalo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; Model (none) -> USBUF02W6; Opis (none) -> Filtr: cyfrowy; line terminator; EMI,dolnoprzepustowy; SOT3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; Producent (none) -> STM; Typ (none) -> SMD
- Y1: footprint Crystals:Crystal_HC49-SD_SMD -> Crystal:Crystal_HC49-U_Vertical; Cena (none) -> 1.6356; Link (none) -> https://www.tme.eu/pl/details/8m-49s-sr/rezonatory-kwarcowe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; Model (none) -> 8M-49S-SR; Opis (none) -> Rezonator: kwarcowy; 8MHz; ±30ppm; 20pF; THT; HC49-S; Producent (none) -> SR PASSIVES; Typ (none) -> THT

Commit message: BOM in KiCad almost finished, genereated NETLIST, create PCB
Parts:
- FB10, FB9: Cena (none) -> 0.2794; Link (none) -> https://www.tme.eu/pl/details/blm21ag102sn1d/ferryty-korali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; Model (none) -> BLM21AG102SN1D; Opis (none) -> Ferryt: koralik; Imp.@ 100MHz: 1000Ω; Montaż: SMD; 0,5A; Ob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; Producent (none) -> MURATA; Typ (none) -> SMD
- J3: Cena (none) -> 2.9560; Link (none) -> https://www.tme.eu/pl/details/2411-02/zlacza-usb-i-ieee1394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; Model (none) -> 2411 02; Opis (none) -> Gniazdo; USB B; na PCB; THT; PIN: 4; kątowe 90°; V: USB 2.0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; Producent (none) -> LUMBERG; Typ (none) -> THT
- J4: Cena (none) -> 1.5839; Link (none) -> https://www.tme.eu/pl/details/t821-1-06-s1/zlacza-idc/amphe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; Model (none) -> T821106A1S100CEU; Opis (none) -> Gniazdo; IDC; męskie; PIN: 6; proste; THT; złocony; 2,54mm;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; Producent (none) -> AMPHENOL; Typ (none) -> THT
- Q1: Cena (none) -> 0.1189; Link (none) -> https://www.tme.eu/pl/details/bc817.215/tranzystory-npn-smd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; Model (none) -> BC817.215; Opis (none) -> Tranzystor: NPN; bipolarny; 45V; 0,5A; 250mW; SOT23; Producent (none) -> NEXPERIA; Typ (none) -> SMD
- R10, R11, R13, R14: Cena (none) -> 0.03622; Link (none) -> https://www.tme.eu/pl/details/smd0603-10k-1%25/rezystory-sm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; Model (none) -> 0603SAF1002T5E; Opis (none) -> Rezystor: thick film; SMD; 0603; 10kΩ; 0,1W; ±1%; -55÷155°C; Producent (none) -> ROYAL OHM; Typ (none) -> SMD
- R12, R15, R16, R17: Cena (none) -> 0.04651; Typ (none) -> SMD
Changed lines of the file:
@@
 F 2 "Resistor_SMD:R_0603_1608Metric" H 3750 6800 50  0001 C CNN
 F 3 "~" H 3750 6800 50  0001 C CNN
+F 4 "0.04651" H 3750 6800 50  0001 C CNN "Cena"
+F 5 "SMD" H 3750 6800 50  0001 C CNN "Typ"
 	1    3750 6800
 	1    0    0    -1
@@
 F 2 "Resistor_SMD:R_0603_1608Metric" H 2650 1750 50  0001 C CNN
 F 3 "~" H 2650 1750 50  0001 C CNN
+F 4 "0.03622" H 2650 1750 50  0001 C CNN "Cena"
+F 5 "https://www.tme.eu/pl/details/smd0603-10k-1%25/rezystory-smd-0603/royal-ohm/0603saf1002t5e/" H 2650 1750 50  0001 C CNN "Link"
+F 6 "0603SAF1002T5E" H 2650 1750 50  0001 C CNN "Model"
+F 7 "Rezystor: thick film; SMD; 0603; 10kΩ; 0,1W; ±1%; -55÷155°C" H 2650 1750 50  0001 C CNN "Opis"
+F 8 "ROYAL OHM" H 2650 1750 50  0001 C CNN "Producent"
+F 9 "SMD" H 2650 1750 50  0001 C CNN "Typ"
 	1    2650 1750
 	0    1    1    0
@@
 F 2 "Resistor_SMD:R_0603_1608Metric" H 2100 1950 50  0001 C CNN
 F 3 "~" H 2100 1950 50  0001 C CNN
+F 4 "0.04651" H 2100 1950 50  0001 C CNN "Cena"
+F 5 "SMD" H 2100 1950 50  0001 C CNN "Typ"
 	1    2100 1950
 	1    0    0    -1
@@
 F 2 "Resistor_SMD:R_0603_1608Metric" H 2650 1400 50  0001 C CNN
 F 3 "~" H 2650 1400 50  0001 C CNN
+F 4 "0.03622" H 2650 1400 50  0001 C CNN "Cena"
+F 5 "https://www.tme.eu/pl/details/smd0603-10k-1%25/rezystory-smd-0603/royal-ohm/0603saf1002t5e/" H 2650 1400 50  0001 C CNN "Link"
+F 6 "0603SAF1002T5E" H 2650 1400 50  0001 C CNN "Model"
+F 7 "Rezystor: thick film; SMD; 0603; 10kΩ; 0,1W; ±1%; -55÷155°C" H 2650 1400 50  0001 C CNN "Opis"
+F 8 "ROYAL OHM" H 2650 1400 50  0001 C CNN "Producent"
+F 9 "SMD" H 2650 1400 50  0001 C CNN "Typ"
 	1    2650 1400
 	1    0    0    -1
@@
 F 2 "Connector_USB:USB_B_OST_USB-B1HSxx_Horizontal" H 7750 1650 50  0001 C CNN
 F 3 " ~" H 7750 1650 50  0001 C CNN
+F 4 "2.9560" H 7600 1700 50  0001 C CNN "Cena"
+F 5 "https://www.tme.eu/pl/details/2411-02/zlacza-usb-i-ieee1394/lumberg/2411-02/" H 7600 1700 50  0001 C CNN "Link"
+F 6 "2411 02" H 7600 1700 50  0001 C CNN "Model"
+F 7 "Gniazdo; USB B; na PCB; THT; PIN: 4; kątowe 90°; V: USB 2.0; biały" H 7600 1700 50  0001 C CNN "Opis"
+F 8 "LUMBERG" H 7600 1700 50  0001 C CNN "Producent"
+F 9 "THT" H 7600 1700 50  0001 C CNN "Typ"
 	1    7600 1700
 	1    0    0    -1
@@
 F 2 "Connector_IDC:IDC-Header_2x03_P2.54mm_Vertical" H 8500 3200 50  0001 C CNN
 F 3 "~" H 8500 3200 50  0001 C CNN
+F 4 "1.5839" H 8500 3200 50  0001 C CNN "Cena"
+F 5 "https://www.tme.eu/pl/details/t821-1-06-s1/zlacza-idc/amphenol/t821106a1s100ceu/" H 8500 3200 50  0001 C CNN "Link"
+F 6 "T821106A1S100CEU" H 8500 3200 50  0001 C CNN "Model"
+F 7 "Gniazdo; IDC; męskie; PIN: 6; proste; THT; złocony; 2,54mm; Układ: 2x3" H 8500 3200 50  0001 C CNN "Opis"
+F 8 "AMPHENOL" H 8500 3200 50  0001 C CNN "Producent"
+F 9 "THT" H 8500 3200 50  0001 C CNN "Typ"
 	1    8500 3200
 	1    0    0    -1
@@
 F 2 "Resistor_SMD:R_0603_1608Metric" V 8030 3100 50  0001 C CNN
 F 3 "~" H 8100 3100 50  0001 C CNN
+F 4 "0.04651" H 8100 3100 50  0001 C CNN "Cena"
+F 5 "SMD" H 8100 3100 50  0001 C CNN "Typ"
 	1    8100 3100
 	0    1    1    0
@@
 F 2 "Inductor_SMD:L_0805_2012Metric" V 8080 5850 50  0001 C CNN
 F 3 "~" H 8150 5850 50  0001 C CNN
+F 4 "0.2794" H 8150 5850 50  0001 C CNN "Cena"
+F 5 "https://www.tme.eu/pl/details/blm21ag102sn1d/ferryty-koraliki/murata/" H 8150 5850 50  0001 C CNN "Link"
+F 6 "BLM21AG102SN1D" H 8150 5850 50  0001 C CNN "Model"
+F 7 "Ferryt: koralik; Imp.@ 100MHz: 1000Ω; Montaż: SMD; 0,5A; Obud: 0805" H 8150 5850 50  0001 C CNN "Opis"
+F 8 "MURATA" H 8150 5850 50  0001 C CNN "Producent"
+F 9 "SMD" H 8150 5850 50  0001 C CNN "Typ"
 	1    8150 5850
 	0    1    1    0
@@
 F 2 "Resistor_SMD:R_0603_1608Metric" V 10030 3550 50  0001 C CNN
 F 3 "~" H 10100 3550 50  0001 C CNN
+F 4 "0.04651" H 10100 3550 50  0001 C CNN "Cena"
+F 5 "SMD" H 10100 3550 50  0001 C CNN "Typ"
 	1    10100 3550
 	1    0    0    -1
@@
 F 2 "Package_TO_SOT_SMD:SOT-23" H 1700 6425 50  0001 L CIN
 F 3 "http://www.fairchildsemi.com/ds/BC/BC817.pdf" H 1500 6500 50  0001 L CNN
+F 4 "0.1189" H 1500 6500 50  0001 C CNN "Cena"
+F 5 "https://www.tme.eu/pl/details/bc817.215/tranzystory-npn-smd/nexperia/" H 1500 6500 50  0001 C CNN "Link"
+F 6 "BC817.215" H 1500 6500 50  0001 C CNN "Model"
+F 7 "Tranzystor: NPN; bipolarny; 45V; 0,5A; 250mW; SOT23" H 1500 6500 50  0001 C CNN "Opis"
+F 8 "NEXPERIA" H 1500 6500 50  0001 C CNN "Producent"
+F 9 "SMD" H 1500 6500 50  0001 C CNN "Typ"
 	1    1500 6500
 	1    0    0    -1
@@
 F 2 "Resistor_SMD:R_0603_1608Metric" V 980 6500 50  0001 C CNN
 F 3 "~" H 1050 6500 50  0001 C CNN
+F 4 "0.03622" H 1050 6500 50  0001 C CNN "Cena"
+F 5 "https://www.tme.eu/pl/details/smd0603-10k-1%25/rezystory-smd-0603/royal-ohm/0603saf1002t5e/" H 1050 6500 50  0001 C CNN "Link"
+F 6 "0603SAF1002T5E" H 1050 6500 50  0001 C CNN "Model"
+F 7 "Rezystor: thick film; SMD; 0603; 10kΩ; 0,1W; ±1%; -55÷155°C" H 1050 6500 50  0001 C CNN "Opis"
+F 8 "ROYAL OHM" H 1050 6500 50  0001 C CNN "Producent"
+F 9 "SMD" H 1050 6500 50  0001 C CNN "Typ"
 	1    1050 6500
 	0    -1   -1   0
@@
 F 2 "Resistor_SMD:R_0603_1608Metric" V 1530 6050 50  0001 C CNN
 F 3 "~" H 1600 6050 50  0001 C CNN
+F 4 "0.03622" H 1600 6050 50  0001 C CNN "Cena"
+F 5 "https://www.tme.eu/pl/details/smd0603-10k-1%25/rezystory-smd-0603/royal-ohm/0603saf1002t5e/" H 1600 6050 50  0001 C CNN "Link"
+F 6 "0603SAF1002T5E" H 1600 6050 50  0001 C CNN "Model"
+F 7 "Rezystor: thick film; SMD; 0603; 10kΩ; 0,1W; ±1%; -55÷155°C" H 1600 6050 50  0001 C CNN "Opis"
+F 8 "ROYAL OHM" H 1600 6050 50  0001 C CNN "Producent"
+F 9 "SMD" H 1600 6050 50  0001 C CNN "Typ"
 	1    1600 6050
 	-1   0    0    1
@@
 F 2 "Inductor_SMD:L_0805_2012Metric" V 8080 5400 50  0001 C CNN
 F 3 "~" H 8150 5400 50  0001 C CNN
+F 4 "0.2794" H 8150 5400 50  0001 C CNN "Cena"
+F 5 "https://www.tme.eu/pl/details/blm21ag102sn1d/ferryty-koraliki/murata/" H 8150 5400 50  0001 C CNN "Link"
+F 6 "BLM21AG102SN1D" H 8150 5400 50  0001 C CNN "Model"
+F 7 "Ferryt: koralik; Imp.@ 100MHz: 1000Ω; Montaż: SMD; 0,5A; Obud: 0805" H 8150 5400 50  0001 C CNN "Opis"
+F 8 "MURATA" H 8150 5400 50  0001 C CNN "Producent"
+F 9 "SMD" H 8150 5400 50  0001 C CNN "Typ"
 	1    8150 5400
 	0    1    1    0
