File: Main Board.kicad_pcb (KiCad board)
At the start: 4 copper layers, 161 x 92 mm, 362 parts, among them J1 Motor Y, J10 CA58SUB-B, J11 PC6 EPSON MAINBOARD, J12 Y AXIS, J13 Z AXIS, J14 LED 1, J15 LED 2, J16 Power Input, J17 VS, J18 12V, J19 5V, J2 Motor Z, J20 3.3V, J21 TABLE SENSOR, J22 INPUT1, J23 INPUT2, J24 PHOTO SENSOR EMITER, J25 PHOTO SENSOR RECEIVER, J26 ANALOG, J27 INPUT3, J28 OUT1, J29 OUT2, J3 USB_B, J30 RELAY, J31 EMERGENCY, J32 EPSON POWER IN, J33 EPSON BOARD POWER, J34 Display, J35 SPI Interface, J36 I2C Interface, J37 LED4, J38 LED3, J39 Key 3, J4 SWD, J40 Key 4, J41 Key 1, J42 Key 2, J43 Encoder, J5 DEBUG, J6 LIMIT Y BACK, J7 LIMIT Y FRONT, J8 LIMIT Z UP, J9 LIMIT Z DOWN, K1 S13-24V-2C, Q1 2N7002K, Q10 2N7002K, Q11 BC817, Q12 BC817, Q13 BC817, Q14 2N7002K, Q15 2N7002K, Q16 2N7002K, Q17 BC817, Q18 2N7002K, Q19 2N7002K, Q2 2N7002K, Q20 2N7002K, Q21 2N7002K, Q3 2N7002K, Q4 2N7002K, Q5 2N7002K, Q6 2N7002K, Q7 2N7002K, Q8 YJS9435A, Q9 2N7002K, U1 TMC2209-LA, U10 74HC2G32, U11 74HC245, U12 SHTC3, U2 TMC2209-LA, U3 STM32F401VETx, U4 USBUF02W6, U5 74HC245, U6 MCP16301, U7 A4403, U8 MCP16301, U9 MCP6002-xSN, Y1 8MHz

Commit message: TMC2209 routing step 2/3
Parts:
- added C87: 10uF, Capacitor_SMD:C_1210_3225Metric, F.Cu at (274.1, 72.6)
- added C88: 1uF, Capacitor_SMD:C_0805_2012Metric, F.Cu at (287.4, 62.4)
- added C89: 0.1uF, Capacitor_SMD:C_0603_1608Metric, F.Cu at (278.9, 71.7)
- added C90: 120uF, Capacitor_THT:CP_Radial_D8.0mm_P3.50mm, F.Cu at (149.9, 87.3)
- added C91: 120uF, Capacitor_THT:CP_Radial_D8.0mm_P3.50mm, F.Cu at (149.9, 69.3)
- added C92: 10uF, Capacitor_SMD:C_1210_3225Metric, F.Cu at (157.7, 86.5)
- added R46: 10Ω, Resistor_SMD:R_0603_1608Metric, F.Cu at (215.2, 63.5)
- C1, C15: value 330uF -> 120uF; footprint Capacitor_THT:CP_Radial_D10.0mm_P5.00mm -> Capacitor_THT:CP_Radial_D8.0mm_P3.50mm
- C2: value 10uF -> 120uF; footprint Capacitor_SMD:C_1210_3225Metric -> Capacitor_THT:CP_Radial_D8.0mm_P3.50mm
- C3: value 1uF -> 120uF; footprint Capacitor_SMD:C_0805_2012Metric -> Capacitor_THT:CP_Radial_D8.0mm_P3.50mm
- C4: value 0.1uF -> 10uF; footprint Capacitor_SMD:C_0603_1608Metric -> Capacitor_SMD:C_1210_3225Metric
- moved R6 96.5 mm to (149.4, 80.3)
- moved C23 96.4 mm to (149.4, 76.3), turned to 180 degrees
- moved C19 95.1 mm to (154.2, 71.8), turned to 90 degrees
- moved R3 92.3 mm to (149.2, 53.8), turned to 180 degrees
- moved R7 91.3 mm to (149.2, 52.3)
- moved C21 84.9 mm to (155.9, 71.8), turned to 270 degrees
- moved U1 84.2 mm to (161.7, 54.5), turned to 270 degrees
- moved C20 77.1 mm to (154.9, 85.8), turned to 270 degrees
- moved C22 76.4 mm to (173.4, 71.8), turned to 90 degrees
- moved C18 73.9 mm to (163.7, 71.8), turned to 90 degrees
- moved C16 73.9 mm to (158.7, 71.2), turned to 90 degrees
- moved FB2 73.0 mm to (179.2, 53.8), turned to 180 degrees
- moved C17 71.8 mm to (161.7, 71.6), turned to 90 degrees
- moved C11 67.5 mm to (175.2, 45.8), turned to 270 degrees
- moved R5 67.1 mm to (171.2, 58.3)
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Connections:
- C20 pad 1: +3V3 -> VCC
- C6 pad 1: +3V3 -> VCC
- R1 pad 1: +3V3 -> VCC
- R3 pad 1: GND -> VCC
- R7 pad 1: GND -> VCC
- U1 pad 15: +3V3 -> VCC
- U1 pad 9: +3V3 -> VCC
- U10 pad 8: +3V3 -> VCC
- U2 pad 15: +3V3 -> VCC

Commit message: Routing almost finished
Parts:
- added R47: 330Ω, Resistor_SMD:R_0603_1608Metric, F.Cu at (130.7, 35.3)
- moved C88 122.6 mm to (164.8, 62.5), turned to 270 degrees
- moved C3 120.4 mm to (158.3, 64.0), turned to 180 degrees
- moved C89 116.4 mm to (162.8, 62.5), turned to 270 degrees
- moved C2 110.3 mm to (160.4, 45.6), turned to 180 degrees
- moved C87 109.7 mm to (167.4, 47.0), turned to 90 degrees
- moved C4 101.6 mm to (167.4, 62.5), turned to 270 degrees
- moved C33 97.3 mm to (129.8, 83.4)
- moved R15 95.0 mm to (169.9, 17.3)
- moved C6 93.9 mm to (157.8, 57.9), turned to 180 degrees
- moved C9 93.4 mm to (157.9, 53.3), turned to 180 degrees
- moved R16 88.5 mm to (169.6, 14.9)
- moved R2 87.2 mm to (157.9, 56.3)
- moved C32 78.4 mm to (111.0, 74.2), turned to 90 degrees
- moved R12 78.1 mm to (136.2, 67.1)
- moved C38 74.1 mm to (129.9, 55.5), turned to 90 degrees
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Connections:
- J3 pad 1: (no net) -> Net-(J3-Pad1)
- J35 pad 4: /HMI/MISO -> Net-(J35-Pad4)
- J5 pad 1: UART_OUT_RX -> UART_OUT_TX
- J5 pad 3: UART_OUT_TX -> UART_OUT_RX
- RN1 pad 1: /Sockets/ZDIR -> /Sockets/LED1_CNT
- RN1 pad 2: /Sockets/ZSTEP -> /Sockets/LED2_CNT
- RN1 pad 3: /Sockets/YDIR -> SPI_SCLK_BUF
- RN1 pad 4: /Sockets/YSTEP -> SPI_MOSI_BUF
- RN2 pad 1: SPI_SCLK_BUF -> /Sockets/YSTEP
- RN2 pad 2: SPI_MOSI_BUF -> /Sockets/YDIR
- RN2 pad 3: /Sockets/LED2_CNT -> /Sockets/ZSTEP
- RN2 pad 4: /Sockets/LED1_CNT -> /Sockets/ZDIR
- RN4 pad 1: SPI_MISO -> Net-(RN4-Pad1)
- U1 pad 10: (no net) -> Net-(U1-Pad10)
- U1 pad 13: (no net) -> Net-(U1-Pad13)
- U1 pad 17: (no net) -> Net-(U1-Pad17)
- U1 pad 20: (no net) -> Net-(U1-Pad20)
- U1 pad 25: (no net) -> Net-(U1-Pad25)
- U1 pad 7: (no net) -> Net-(U1-Pad7)
- U11 pad 11: Net-(RN4-Pad8) -> Net-(U11-Pad11)
- U11 pad 4: LCD_DB4 -> LCD_DB7
- U11 pad 5: LCD_DB5 -> LCD_DB6
- U11 pad 6: LCD_DB6 -> LCD_DB5
- U11 pad 7: LCD_DB7 -> LCD_DB4
- U11 pad 9: /HMI/MISO -> Net-(U11-Pad9)
- U12 pad 5: (no net) -> Net-(U12-Pad5)
- U2 pad 10: (no net) -> Net-(U2-Pad10)
- U2 pad 13: (no net) -> Net-(U2-Pad13)
- U2 pad 17: (no net) -> Net-(U2-Pad17)
- U2 pad 20: (no net) -> Net-(U2-Pad20)
- U2 pad 25: (no net) -> Net-(U2-Pad25)
- U2 pad 7: (no net) -> Net-(U2-Pad7)
- U2 pad 9: (no net) -> Net-(U2-Pad9)
- U3 pad 15: (no net) -> Net-(U3-Pad15)
- U3 pad 42: (no net) -> Net-(U3-Pad42)
- U3 pad 43: (no net) -> Net-(U3-Pad43)
- U3 pad 44: (no net) -> Net-(U3-Pad44)
- U3 pad 45: (no net) -> Net-(U3-Pad45)
- U3 pad 46: (no net) -> Net-(U3-Pad46)
- U3 pad 47: (no net) -> Net-(U3-Pad47)
- U3 pad 51: (no net) -> Net-(U3-Pad51)
- U3 pad 59: (no net) -> Net-(U3-Pad59)
- U3 pad 61: (no net) -> Net-(U3-Pad61)
- U3 pad 62: (no net) -> Net-(U3-Pad62)
- U3 pad 65: (no net) -> Net-(U3-Pad65)
- U3 pad 68: (no net) -> Net-(U3-Pad68)
- U3 pad 69: (no net) -> Net-(U3-Pad69)
- U3 pad 8: (no net) -> Net-(U3-Pad8)
- U3 pad 9: (no net) -> Net-(U3-Pad9)
- U5 pad 2: Y_STEP -> SPI_MOSI
- U5 pad 3: Y_DIR -> SPI_SCLK
- U5 pad 4: Z_STEP -> LED2_CONTROL
- U5 pad 5: Z_DIR -> LED1_CONTROL
- U5 pad 6: LED1_CONTROL -> Z_DIR
- U5 pad 7: LED2_CONTROL -> Z_STEP
- U5 pad 8: SPI_MOSI -> Y_DIR
- U5 pad 9: SPI_SCLK -> Y_STEP
Routing:
- net LIMIT_Y_BACK: track 0.00 -> 76.7 mm
- net Z_STEP: track 0.00 -> 73.1 mm, vias 0 -> 3
- net Z_DIR: track 0.00 -> 72.7 mm, vias 0 -> 3
- net Y_DIR: track 0.00 -> 68.5 mm, vias 0 -> 3
- net UART_OUT_TX: track 0.00 -> 68.0 mm, vias 0 -> 1
- net LIMIT_Z_DOWN: track 0.00 -> 67.6 mm
- net UART_OUT_RX: track 0.00 -> 66.4 mm, vias 0 -> 1
- net Y_STEP: track 0.00 -> 65.9 mm, vias 0 -> 3
- net LIMIT_Y_FRONT: track 0.00 -> 63.9 mm
- net LCD_RS: track 0.00 -> 58.9 mm, vias 0 -> 2
- net I2C_SCL: track 0.00 -> 56.7 mm, vias 0 -> 2
- net I2C_SDA: track 0.00 -> 54.6 mm, vias 0 -> 2
- net LCD_E: track 0.00 -> 54.1 mm
- net LCD_DB7: track 0.00 -> 53.2 mm
- net LCD_DB6: track 0.00 -> 52.3 mm
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- added copper zone on F.Cu, net Net-(C10-Pad1)
- added copper zone on F.Cu, net Net-(C11-Pad2)
- added copper zone on F.Cu, net Net-(C12-Pad1)
- added copper zone on F.Cu, net Net-(C13-Pad2)
- added copper zone on In2.Cu, net Net-(C13-Pad2)
- added copper zone on F.Cu, net Net-(C14-Pad1)
- added copper zone on In2.Cu, net Net-(C14-Pad1)
- added copper zone on In2.Cu, net Net-(C27-Pad2)
- added copper zone on In2.Cu, net Net-(C28-Pad1)
- added copper zone on F.Cu, net Net-(C8-Pad1)
- added copper zone on F.Cu, net Net-(FB1-Pad2)
- added copper zone on F.Cu, net Net-(FB2-Pad2)
- added copper zone on F.Cu, net Net-(FB3-Pad2)
- added copper zone on F.Cu, net Net-(FB4-Pad2)
