File: Emergency.sch (KiCad schematic (older format))
At the start: 18 parts, among them J31 EMERGENCY, J32 EPSON POWER IN, J33 EPSON BOARD POWER, K1 S13-24V-2C, Q17 BC817, U10 74HC2G32

Commit message: Updated BOM on schematics
Parts:
- C77: Cena 0.05563 -> 0.07894; Dielektryk (none) -> X7R; Link https://www.tme.eu/pl/details/cl10b102kb8nnnc/kondensatory-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 -> https://www.tme.eu/pl/details/cl10b104kb8nnnc/kondensatory-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; Model CL10B102KB8NNNC -> CL10B104KB8NNNC; Napięcie (none) -> 50V; Opis Kondensator: ceramiczny; MLCC; 1nF; 50V; X7R; ±10%; SMD; 06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 -> Kondensator: ceramiczny; MLCC; 100nF; 50V; X7R; ±10%; SMD; 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
- R88: Cena (none) -> 0.045; Link (none) -> https://www.tme.eu/pl/details/smd0805-0r/rezystory-smd-0805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; Model (none) -> 0805S8J0000T5E; Opis (none) -> Rezystor: thick film; SMD; 0805; 0Ω; 0,125W; ±5%; -55÷125°C; Producent (none) -> ROYAL OHM; Typ (none) -> SMD
- R91, R92, R94, R95: Link (none) -> https://www.tme.eu/pl/details/smd0603-100k-1%25/rezystory-s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; Model (none) -> 0603SAF1003T5E; Opis (none) -> Rezystor: thick film; SMD; 0603; 100kΩ; 0,1W; ±1%; -55÷155°C; Producent (none) -> ROYAL OHM
- R93: Link https://www.tme.eu/pl/details/smd0603-1k-1%25/rezystory-smd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 -> https://www.tme.eu/pl/details/smd0603-47k/rezystory-smd-060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; Model 0603SAF1001T5E -> 0603SAJ0473T5E; Opis Rezystor: thick film; SMD; 0603; 1kΩ; 0,1W; ±1%; -55÷155°C -> Rezystor: thick film; SMD; 0603; 47kΩ; 0,1W; ±5%; -55÷155°C
Changed lines of the file:
@@
 F 4 "0.04651" H 5900 2350 50  0001 C CNN "Cena"
 F 5 "SMD" H 5900 2350 50  0001 C CNN "Typ"
+F 6 "https://www.tme.eu/pl/details/smd0603-100k-1%25/rezystory-smd-0603/royal-ohm/0603saf1003t5e/" H 5900 2350 50  0001 C CNN "Link"
+F 7 "0603SAF1003T5E" H 5900 2350 50  0001 C CNN "Model"
+F 8 "Rezystor: thick film; SMD; 0603; 100kΩ; 0,1W; ±1%; -55÷155°C" H 5900 2350 50  0001 C CNN "Opis"
+F 9 "ROYAL OHM" H 5900 2350 50  0001 C CNN "Producent"
 	1    5900 2350
 	0    1    1    0
@@
 F 3 "~" H 6650 1900 50  0001 C CNN
 F 4 "0.04651" H 6650 1900 50  0001 C CNN "Cena"
-F 5 "https://www.tme.eu/pl/details/smd0603-1k-1%25/rezystory-smd-0603/royal-ohm/0603saf1001t5e/" H 6650 1900 50  0001 C CNN "Link"
-F 6 "0603SAF1001T5E" H 6650 1900 50  0001 C CNN "Model"
-F 7 "Rezystor: thick film; SMD; 0603; 1kΩ; 0,1W; ±1%; -55÷155°C" H 6650 1900 50  0001 C CNN "Opis"
+F 5 "https://www.tme.eu/pl/details/smd0603-47k/rezystory-smd-0603/royal-ohm/0603saj0473t5e/" H 6650 1900 50  0001 C CNN "Link"
+F 6 "0603SAJ0473T5E" H 6650 1900 50  0001 C CNN "Model"
+F 7 "Rezystor: thick film; SMD; 0603; 47kΩ; 0,1W; ±5%; -55÷155°C" H 6650 1900 50  0001 C CNN "Opis"
 F 8 "ROYAL OHM" H 6650 1900 50  0001 C CNN "Producent"
 F 9 "SMD" H 6650 1900 50  0001 C CNN "Typ"
@@
 F 4 "0.04651" H 7650 3950 50  0001 C CNN "Cena"
 F 5 "SMD" H 7650 3950 50  0001 C CNN "Typ"
+F 6 "https://www.tme.eu/pl/details/smd0603-100k-1%25/rezystory-smd-0603/royal-ohm/0603saf1003t5e/" H 7650 3950 50  0001 C CNN "Link"
+F 7 "0603SAF1003T5E" H 7650 3950 50  0001 C CNN "Model"
+F 8 "Rezystor: thick film; SMD; 0603; 100kΩ; 0,1W; ±1%; -55÷155°C" H 7650 3950 50  0001 C CNN "Opis"
+F 9 "ROYAL OHM" H 7650 3950 50  0001 C CNN "Producent"
 	1    7650 3950
 	1    0    0    -1
@@
 F 4 "0.04651" H 7650 3200 50  0001 C CNN "Cena"
 F 5 "SMD" H 7650 3200 50  0001 C CNN "Typ"
+F 6 "https://www.tme.eu/pl/details/smd0603-100k-1%25/rezystory-smd-0603/royal-ohm/0603saf1003t5e/" H 7650 3200 50  0001 C CNN "Link"
+F 7 "0603SAF1003T5E" H 7650 3200 50  0001 C CNN "Model"
+F 8 "Rezystor: thick film; SMD; 0603; 100kΩ; 0,1W; ±1%; -55÷155°C" H 7650 3200 50  0001 C CNN "Opis"
+F 9 "ROYAL OHM" H 7650 3200 50  0001 C CNN "Producent"
 	1    7650 3200
 	1    0    0    -1
@@
 F 2 "Capacitor_SMD:C_0603_1608Metric" H 7200 2350 50  0001 C CNN
 F 3 "~" H 7200 2350 50  0001 C CNN
-F 4 "0.05563" H 7200 2350 50  0001 C CNN "Cena"
-F 5 "https://www.tme.eu/pl/details/cl10b102kb8nnnc/kondensatory-mlcc-smd-0603/samsung/" H 7200 2350 50  0001 C CNN "Link"
-F 6 "CL10B102KB8NNNC" H 7200 2350 50  0001 C CNN "Model"
-F 7 "Kondensator: ceramiczny; MLCC; 1nF; 50V; X7R; ±10%; SMD; 0603" H 7200 2350 50  0001 C CNN "Opis"
+F 4 "0.07894" H 7200 2350 50  0001 C CNN "Cena"
+F 5 "https://www.tme.eu/pl/details/cl10b104kb8nnnc/kondensatory-mlcc-smd-0603/samsung/" H 7200 2350 50  0001 C CNN "Link"
+F 6 "CL10B104KB8NNNC" H 7200 2350 50  0001 C CNN "Model"
+F 7 "Kondensator: ceramiczny; MLCC; 100nF; 50V; X7R; ±10%; SMD; 0603" H 7200 2350 50  0001 C CNN "Opis"
 F 8 "SAMSUNG" H 7200 2350 50  0001 C CNN "Producent"
 F 9 "SMD" H 7200 2350 50  0001 C CNN "Typ"
+F 10 "X7R" H 7200 2350 50  0001 C CNN "Dielektryk"
+F 11 "50V" H 7200 2350 50  0001 C CNN "Napięcie"
 	1    7200 2350
 	1    0    0    -1
@@
 F 2 "Resistor_SMD:R_0805_2012Metric" V 3330 3800 50  0001 C CNN
 F 3 "~" H 3400 3800 50  0001 C CNN
+F 4 "0.045" H 3400 3800 50  0001 C CNN "Cena"
+F 5 "https://www.tme.eu/pl/details/smd0805-0r/rezystory-smd-0805/royal-ohm/0805s8j0000t5e/" H 3400 3800 50  0001 C CNN "Link"
+F 6 "0805S8J0000T5E" H 3400 3800 50  0001 C CNN "Model"
+F 7 "Rezystor: thick film; SMD; 0805; 0Ω; 0,125W; ±5%; -55÷125°C" H 3400 3800 50  0001 C CNN "Opis"
+F 8 "ROYAL OHM" H 3400 3800 50  0001 C CNN "Producent"
+F 9 "SMD" H 3400 3800 50  0001 C CNN "Typ"
 	1    3400 3800
 	0    1    1    0
@@
 F 4 "0.04651" H 6250 2550 50  0001 C CNN "Cena"
 F 5 "SMD" H 6250 2550 50  0001 C CNN "Typ"
+F 6 "https://www.tme.eu/pl/details/smd0603-100k-1%25/rezystory-smd-0603/royal-ohm/0603saf1003t5e/" H 6250 2550 50  0001 C CNN "Link"
+F 7 "0603SAF1003T5E" H 6250 2550 50  0001 C CNN "Model"
+F 8 "Rezystor: thick film; SMD; 0603; 100kΩ; 0,1W; ±1%; -55÷155°C" H 6250 2550 50  0001 C CNN "Opis"
+F 9 "ROYAL OHM" H 6250 2550 50  0001 C CNN "Producent"
 	1    6250 2550
 	1    0    0    -1
