File: Sockets 2.sch (KiCad schematic (older format))
At the start: 70 parts, among them J21 TABLE SENSOR, J22 INPUT1, J23 INPUT2, J24 PHOTO SENSOR EMITER, J25 PHOTO SENSOR RECEIVER, J26 ANALOG, J27 INPUT3, J28 OUT1, J29 OUT2, J30 RELAY, Q10 2N7002K, Q11 BC817, Q12 BC817, Q13 BC817, Q14 2N7002K, Q15 2N7002K, Q16 2N7002K, Q9 2N7002K, U9 MCP6002-xSN

Commit message: Updated BOM on schematics
Parts:
- C67, C68, C69, C70, C75: Cena 0.05563 -> 0.07894; Dielektryk (none) -> X7R; Link https://www.tme.eu/pl/details/cl10b102kb8nnnc/kondensatory-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 -> https://www.tme.eu/pl/details/cl10b104kb8nnnc/kondensatory-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; Model CL10B102KB8NNNC -> CL10B104KB8NNNC; Napięcie (none) -> 50V; Opis Kondensator: ceramiczny; MLCC; 1nF; 50V; X7R; ±10%; SMD; 06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 -> Kondensator: ceramiczny; MLCC; 100nF; 50V; X7R; ±10%; SMD; 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
- C84: Cena 0.05982 -> 0.07894; Dielektryk (none) -> X7R; Link (none) -> https://www.tme.eu/pl/details/cl10b104kb8nnnc/kondensatory-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; Model CL10B104KB8NNNC -> CL10B104KB8NNNC; Opis (none) -> Kondensator: ceramiczny; MLCC; 100nF; 50V; X7R; ±10%; SMD; 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
- R64, R67, R68, R69, R82, R83: Link (none) -> https://www.tme.eu/pl/details/smd0603-100k-1%25/rezystory-s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; Model (none) -> 0603SAF1003T5E; Opis (none) -> Rezystor: thick film; SMD; 0603; 100kΩ; 0,1W; ±1%; -55÷155°C; Producent (none) -> ROYAL OHM
Changed lines of the file:
@@
 F 4 "0.04651" H 2100 1700 50  0001 C CNN "Cena"
 F 5 "SMD" H 2100 1700 50  0001 C CNN "Typ"
+F 6 "https://www.tme.eu/pl/details/smd0603-100k-1%25/rezystory-smd-0603/royal-ohm/0603saf1003t5e/" H 2100 1700 50  0001 C CNN "Link"
+F 7 "0603SAF1003T5E" H 2100 1700 50  0001 C CNN "Model"
+F 8 "Rezystor: thick film; SMD; 0603; 100kΩ; 0,1W; ±1%; -55÷155°C" H 2100 1700 50  0001 C CNN "Opis"
+F 9 "ROYAL OHM" H 2100 1700 50  0001 C CNN "Producent"
 	1    2100 1700
 	0    1    1    0
@@
 F 2 "Capacitor_SMD:C_0603_1608Metric" H 3588 1550 50  0001 C CNN
 F 3 "~" H 3550 1700 50  0001 C CNN
-F 4 "0.05563" H 3550 1700 50  0001 C CNN "Cena"
-F 5 "https://www.tme.eu/pl/details/cl10b102kb8nnnc/kondensatory-mlcc-smd-0603/samsung/" H 3550 1700 50  0001 C CNN "Link"
-F 6 "CL10B102KB8NNNC" H 3550 1700 50  0001 C CNN "Model"
-F 7 "Kondensator: ceramiczny; MLCC; 1nF; 50V; X7R; ±10%; SMD; 0603" H 3550 1700 50  0001 C CNN "Opis"
+F 4 "0.07894" H 3550 1700 50  0001 C CNN "Cena"
+F 5 "https://www.tme.eu/pl/details/cl10b104kb8nnnc/kondensatory-mlcc-smd-0603/samsung/" H 3550 1700 50  0001 C CNN "Link"
+F 6 "CL10B104KB8NNNC" H 3550 1700 50  0001 C CNN "Model"
+F 7 "Kondensator: ceramiczny; MLCC; 100nF; 50V; X7R; ±10%; SMD; 0603" H 3550 1700 50  0001 C CNN "Opis"
 F 8 "SAMSUNG" H 3550 1700 50  0001 C CNN "Producent"
 F 9 "SMD" H 3550 1700 50  0001 C CNN "Typ"
+F 10 "X7R" H 3550 1700 50  0001 C CNN "Dielektryk"
+F 11 "50V" H 3550 1700 50  0001 C CNN "Napięcie"
 	1    3550 1700
 	1    0    0    -1
@@
 F 4 "0.04651" H 2350 3850 50  0001 C CNN "Cena"
 F 5 "SMD" H 2350 3850 50  0001 C CNN "Typ"
+F 6 "https://www.tme.eu/pl/details/smd0603-100k-1%25/rezystory-smd-0603/royal-ohm/0603saf1003t5e/" H 2350 3850 50  0001 C CNN "Link"
+F 7 "0603SAF1003T5E" H 2350 3850 50  0001 C CNN "Model"
+F 8 "Rezystor: thick film; SMD; 0603; 100kΩ; 0,1W; ±1%; -55÷155°C" H 2350 3850 50  0001 C CNN "Opis"
+F 9 "ROYAL OHM" H 2350 3850 50  0001 C CNN "Producent"
 	1    2350 3850
 	0    1    1    0
@@
 F 2 "Capacitor_SMD:C_0603_1608Metric" H 3838 3700 50  0001 C CNN
 F 3 "~" H 3800 3850 50  0001 C CNN
-F 4 "0.05563" H 3800 3850 50  0001 C CNN "Cena"
-F 5 "https://www.tme.eu/pl/details/cl10b102kb8nnnc/kondensatory-mlcc-smd-0603/samsung/" H 3800 3850 50  0001 C CNN "Link"
-F 6 "CL10B102KB8NNNC" H 3800 3850 50  0001 C CNN "Model"
-F 7 "Kondensator: ceramiczny; MLCC; 1nF; 50V; X7R; ±10%; SMD; 0603" H 3800 3850 50  0001 C CNN "Opis"
+F 4 "0.07894" H 3800 3850 50  0001 C CNN "Cena"
+F 5 "https://www.tme.eu/pl/details/cl10b104kb8nnnc/kondensatory-mlcc-smd-0603/samsung/" H 3800 3850 50  0001 C CNN "Link"
+F 6 "CL10B104KB8NNNC" H 3800 3850 50  0001 C CNN "Model"
+F 7 "Kondensator: ceramiczny; MLCC; 100nF; 50V; X7R; ±10%; SMD; 0603" H 3800 3850 50  0001 C CNN "Opis"
 F 8 "SAMSUNG" H 3800 3850 50  0001 C CNN "Producent"
 F 9 "SMD" H 3800 3850 50  0001 C CNN "Typ"
+F 10 "X7R" H 3800 3850 50  0001 C CNN "Dielektryk"
+F 11 "50V" H 3800 3850 50  0001 C CNN "Napięcie"
 	1    3800 3850
 	1    0    0    -1
@@
 F 2 "Capacitor_SMD:C_0603_1608Metric" H 2988 6950 50  0001 C CNN
 F 3 "~" H 2950 7100 50  0001 C CNN
-F 4 "0.05563" H 2950 7100 50  0001 C CNN "Cena"
-F 5 "https://www.tme.eu/pl/details/cl10b102kb8nnnc/kondensatory-mlcc-smd-0603/samsung/" H 2950 7100 50  0001 C CNN "Link"
-F 6 "CL10B102KB8NNNC" H 2950 7100 50  0001 C CNN "Model"
-F 7 "Kondensator: ceramiczny; MLCC; 1nF; 50V; X7R; ±10%; SMD; 0603" H 2950 7100 50  0001 C CNN "Opis"
+F 4 "0.07894" H 2950 7100 50  0001 C CNN "Cena"
+F 5 "https://www.tme.eu/pl/details/cl10b104kb8nnnc/kondensatory-mlcc-smd-0603/samsung/" H 2950 7100 50  0001 C CNN "Link"
+F 6 "CL10B104KB8NNNC" H 2950 7100 50  0001 C CNN "Model"
+F 7 "Kondensator: ceramiczny; MLCC; 100nF; 50V; X7R; ±10%; SMD; 0603" H 2950 7100 50  0001 C CNN "Opis"
 F 8 "SAMSUNG" H 2950 7100 50  0001 C CNN "Producent"
 F 9 "SMD" H 2950 7100 50  0001 C CNN "Typ"
+F 10 "X7R" H 2950 7100 50  0001 C CNN "Dielektryk"
+F 11 "50V" H 2950 7100 50  0001 C CNN "Napięcie"
 	1    2950 7100
 	1    0    0    -1
@@
 F 2 "Capacitor_SMD:C_0603_1608Metric" H 2988 5450 50  0001 C CNN
 F 3 "~" H 2950 5600 50  0001 C CNN
-F 4 "0.05563" H 2950 5600 50  0001 C CNN "Cena"
-F 5 "https://www.tme.eu/pl/details/cl10b102kb8nnnc/kondensatory-mlcc-smd-0603/samsung/" H 2950 5600 50  0001 C CNN "Link"
-F 6 "CL10B102KB8NNNC" H 2950 5600 50  0001 C CNN "Model"
-F 7 "Kondensator: ceramiczny; MLCC; 1nF; 50V; X7R; ±10%; SMD; 0603" H 2950 5600 50  0001 C CNN "Opis"
+F 4 "0.07894" H 2950 5600 50  0001 C CNN "Cena"
+F 5 "https://www.tme.eu/pl/details/cl10b104kb8nnnc/kondensatory-mlcc-smd-0603/samsung/" H 2950 5600 50  0001 C CNN "Link"
+F 6 "CL10B104KB8NNNC" H 2950 5600 50  0001 C CNN "Model"
+F 7 "Kondensator: ceramiczny; MLCC; 100nF; 50V; X7R; ±10%; SMD; 0603" H 2950 5600 50  0001 C CNN "Opis"
 F 8 "SAMSUNG" H 2950 5600 50  0001 C CNN "Producent"
 F 9 "SMD" H 2950 5600 50  0001 C CNN "Typ"
+F 10 "X7R" H 2950 5600 50  0001 C CNN "Dielektryk"
+F 11 "50V" H 2950 5600 50  0001 C CNN "Napięcie"
 	1    2950 5600
 	1    0    0    -1
@@
 F 4 "0.04651" H 6100 1650 50  0001 C CNN "Cena"
 F 5 "SMD" H 6100 1650 50  0001 C CNN "Typ"
+F 6 "https://www.tme.eu/pl/details/smd0603-100k-1%25/rezystory-smd-0603/royal-ohm/0603saf1003t5e/" H 6100 1650 50  0001 C CNN "Link"
+F 7 "0603SAF1003T5E" H 6100 1650 50  0001 C CNN "Model"
+F 8 "Rezystor: thick film; SMD; 0603; 100kΩ; 0,1W; ±1%; -55÷155°C" H 6100 1650 50  0001 C CNN "Opis"
+F 9 "ROYAL OHM" H 6100 1650 50  0001 C CNN "Producent"
 	1    6100 1650
 	0    1    1    0
@@
 F 2 "Capacitor_SMD:C_0603_1608Metric" H 7588 1500 50  0001 C CNN
 F 3 "~" H 7550 1650 50  0001 C CNN
-F 4 "0.05563" H 7550 1650 50  0001 C CNN "Cena"
-F 5 "https://www.tme.eu/pl/details/cl10b102kb8nnnc/kondensatory-mlcc-smd-0603/samsung/" H 7550 1650 50  0001 C CNN "Link"
-F 6 "CL10B102KB8NNNC" H 7550 1650 50  0001 C CNN "Model"
-F 7 "Kondensator: ceramiczny; MLCC; 1nF; 50V; X7R; ±10%; SMD; 0603" H 7550 1650 50  0001 C CNN "Opis"
+F 4 "0.07894" H 7550 1650 50  0001 C CNN "Cena"
+F 5 "https://www.tme.eu/pl/details/cl10b104kb8nnnc/kondensatory-mlcc-smd-0603/samsung/" H 7550 1650 50  0001 C CNN "Link"
+F 6 "CL10B104KB8NNNC" H 7550 1650 50  0001 C CNN "Model"
+F 7 "Kondensator: ceramiczny; MLCC; 100nF; 50V; X7R; ±10%; SMD; 0603" H 7550 1650 50  0001 C CNN "Opis"
 F 8 "SAMSUNG" H 7550 1650 50  0001 C CNN "Producent"
 F 9 "SMD" H 7550 1650 50  0001 C CNN "Typ"
+F 10 "X7R" H 7550 1650 50  0001 C CNN "Dielektryk"
+F 11 "50V" H 7550 1650 50  0001 C CNN "Napięcie"
 	1    7550 1650
 	1    0    0    -1
@@
 F 4 "0.04651" H 2350 1900 50  0001 C CNN "Cena"
 F 5 "SMD" H 2350 1900 50  0001 C CNN "Typ"
+F 6 "https://www.tme.eu/pl/details/smd0603-100k-1%25/rezystory-smd-0603/royal-ohm/0603saf1003t5e/" H 2350 1900 50  0001 C CNN "Link"
+F 7 "0603SAF1003T5E" H 2350 1900 50  0001 C CNN "Model"
+F 8 "Rezystor: thick film; SMD; 0603; 100kΩ; 0,1W; ±1%; -55÷155°C" H 2350 1900 50  0001 C CNN "Opis"
+F 9 "ROYAL OHM" H 2350 1900 50  0001 C CNN "Producent"
 	1    2350 1900
 	1    0    0    -1
@@
 F 4 "0.04651" H 2600 4050 50  0001 C CNN "Cena"
 F 5 "SMD" H 2600 4050 50  0001 C CNN "Typ"
+F 6 "https://www.tme.eu/pl/details/smd0603-100k-1%25/rezystory-smd-0603/royal-ohm/0603saf1003t5e/" H 2600 4050 50  0001 C CNN "Link"
+F 7 "0603SAF1003T5E" H 2600 4050 50  0001 C CNN "Model"
+F 8 "Rezystor: thick film; SMD; 0603; 100kΩ; 0,1W; ±1%; -55÷155°C" H 2600 4050 50  0001 C CNN "Opis"
+F 9 "ROYAL OHM" H 2600 4050 50  0001 C CNN "Producent"
 	1    2600 4050
 	1    0    0    -1
@@
 F 4 "0.04651" H 6350 1850 50  0001 C CNN "Cena"
 F 5 "SMD" H 6350 1850 50  0001 C CNN "Typ"
+F 6 "https://www.tme.eu/pl/details/smd0603-100k-1%25/rezystory-smd-0603/royal-ohm/0603saf1003t5e/" H 6350 1850 50  0001 C CNN "Link"
+F 7 "0603SAF1003T5E" H 6350 1850 50  0001 C CNN "Model"
+F 8 "Rezystor: thick film; SMD; 0603; 100kΩ; 0,1W; ±1%; -55÷155°C" H 6350 1850 50  0001 C CNN "Opis"
+F 9 "ROYAL OHM" H 6350 1850 50  0001 C CNN "Producent"
 	1    6350 1850
 	1    0    0    -1
@@
 F 2 "Capacitor_SMD:C_0603_1608Metric" H 6800 4350 50  0001 C CNN
 F 3 "~" H 6800 4350 50  0001 C CNN
-F 4 "0.05982" H 6800 4350 50  0001 C CNN "Cena"
-F 5 "CL10B104KB8NNNC " H 6800 4350 50  0001 C CNN "Model"
+F 4 "0.07894" H 6800 4350 50  0001 C CNN "Cena"
+F 5 "CL10B104KB8NNNC" H 6800 4350 50  0001 C CNN "Model"
 F 6 "50V" H 6800 4350 50  0001 C CNN "Napięcie"
 F 7 "SAMSUNG" H 6800 4350 50  0001 C CNN "Producent"
 F 8 "10%" H 6800 4350 50  0001 C CNN "Tolerancja"
 F 9 "SMD" H 6800 4350 50  0001 C CNN "Typ"
+F 10 "X7R" H 6800 4350 50  0001 C CNN "Dielektryk"
+F 11 "https://www.tme.eu/pl/details/cl10b104kb8nnnc/kondensatory-mlcc-smd-0603/samsung/" H 6800 4350 50  0001 C CNN "Link"
+F 12 "Kondensator: ceramiczny; MLCC; 100nF; 50V; X7R; ±10%; SMD; 0603" H 6800 4350 50  0001 C CNN "Opis"
 	1    6800 4350
 	1    0    0    -1
