File: Sockets.sch (KiCad schematic (older format))
At the start: 61 parts, among them J10 CA58SUB-B, J11 PC6 EPSON MAINBOARD, J12 Y AXIS, J13 Z AXIS, J14 LED 1, J15 LED 2, J6 LIMIT Y BACK, J7 LIMIT Y FRONT, J8 LIMIT Z UP, J9 LIMIT Z DOWN, Q1 2N7002K, Q2 2N7002K, Q3 2N7002K, Q4 2N7002K, Q5 2N7002K, Q6 2N7002K, Q7 2N7002K, U5 74HC245

Commit message: Updated BOM on schematics
Parts:
- C43, C44, C45, C46, C48: Cena 0.05563 -> 0.07894; Dielektryk (none) -> X7R; Link https://www.tme.eu/pl/details/cl10b102kb8nnnc/kondensatory-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 -> https://www.tme.eu/pl/details/cl10b104kb8nnnc/kondensatory-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; Model CL10B102KB8NNNC -> CL10B104KB8NNNC; Napięcie (none) -> 50V; Opis Kondensator: ceramiczny; MLCC; 1nF; 50V; X7R; ±10%; SMD; 06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 -> Kondensator: ceramiczny; MLCC; 100nF; 50V; X7R; ±10%; SMD; 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
- C47: Cena 0.05982 -> 0.07894; Link (none) -> https://www.tme.eu/pl/details/cl10b104kb8nnnc/kondensatory-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; Model CL10B104KB8NNNC -> CL10B104KB8NNNC; Opis (none) -> Kondensator: ceramiczny; MLCC; 100nF; 50V; X7R; ±10%; SMD; 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
- R32, R33, R34, R36, R37: Link (none) -> https://www.tme.eu/pl/details/0603saj0000t5e/rezystory-smd-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; Model (none) -> 0603SAJ0000T5E; Opis (none) -> Rezystor: thick film; SMD; 0603; 0Ω; 0,1W; ±5%; -55÷155°C; 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; Producent (none) -> ROYAL OHM
- R39: Link (none) -> https://www.tme.eu/pl/details/smd0603-100k-1%25/rezystory-s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; Model (none) -> 0603SAF1003T5E; Opis (none) -> Rezystor: thick film; SMD; 0603; 100kΩ; 0,1W; ±1%; -55÷155°C; Producent (none) -> ROYAL OHM; Typ (none) -> SMD
Changed lines of the file:
@@
 F 4 "0.04651" H 6350 1300 50  0001 C CNN "Cena"
 F 5 "SMD" H 6350 1300 50  0001 C CNN "Typ"
+F 6 "https://www.tme.eu/pl/details/0603saj0000t5e/rezystory-smd-0603/royal-ohm/" H 6350 1300 50  0001 C CNN "Link"
+F 7 "0603SAJ0000T5E" H 6350 1300 50  0001 C CNN "Model"
+F 8 "Rezystor: thick film; SMD; 0603; 0Ω; 0,1W; ±5%; -55÷155°C; 400ppm/°C" H 6350 1300 50  0001 C CNN "Opis"
+F 9 "ROYAL OHM" H 6350 1300 50  0001 C CNN "Producent"
 	1    6350 1300
 	0    -1   -1   0
@@
 F 4 "0.04651" H 6350 1500 50  0001 C CNN "Cena"
 F 5 "SMD" H 6350 1500 50  0001 C CNN "Typ"
+F 6 "https://www.tme.eu/pl/details/0603saj0000t5e/rezystory-smd-0603/royal-ohm/" H 6350 1500 50  0001 C CNN "Link"
+F 7 "0603SAJ0000T5E" H 6350 1500 50  0001 C CNN "Model"
+F 8 "Rezystor: thick film; SMD; 0603; 0Ω; 0,1W; ±5%; -55÷155°C; 400ppm/°C" H 6350 1500 50  0001 C CNN "Opis"
+F 9 "ROYAL OHM" H 6350 1500 50  0001 C CNN "Producent"
 	1    6350 1500
 	0    -1   -1   0
@@
 F 2 "Capacitor_SMD:C_0603_1608Metric" H 5388 4900 50  0001 C CNN
 F 3 "~" H 5350 5050 50  0001 C CNN
-F 4 "0.05982" H 5350 5050 50  0001 C CNN "Cena"
+F 4 "0.07894" H 5350 5050 50  0001 C CNN "Cena"
 F 5 "X7R" H 5350 5050 50  0001 C CNN "Dielektryk"
-F 6 "CL10B104KB8NNNC " H 5350 5050 50  0001 C CNN "Model"
+F 6 "CL10B104KB8NNNC" H 5350 5050 50  0001 C CNN "Model"
 F 7 "50V" H 5350 5050 50  0001 C CNN "Napięcie"
 F 8 "SAMSUNG" H 5350 5050 50  0001 C CNN "Producent"
 F 9 "10%" H 5350 5050 50  0001 C CNN "Tolerancja"
 F 10 "SMD" H 5350 5050 50  0001 C CNN "Typ"
+F 11 "https://www.tme.eu/pl/details/cl10b104kb8nnnc/kondensatory-mlcc-smd-0603/samsung/" H 5350 5050 50  0001 C CNN "Link"
+F 12 "Kondensator: ceramiczny; MLCC; 100nF; 50V; X7R; ±10%; SMD; 0603" H 5350 5050 50  0001 C CNN "Opis"
 	1    5350 5050
 	1    0    0    -1
@@
 F 2 "Capacitor_SMD:C_0603_1608Metric" H 2938 1550 50  0001 C CNN
 F 3 "~" H 2900 1700 50  0001 C CNN
-F 4 "0.05563" H 2900 1700 50  0001 C CNN "Cena"
-F 5 "https://www.tme.eu/pl/details/cl10b102kb8nnnc/kondensatory-mlcc-smd-0603/samsung/" H 2900 1700 50  0001 C CNN "Link"
-F 6 "CL10B102KB8NNNC" H 2900 1700 50  0001 C CNN "Model"
-F 7 "Kondensator: ceramiczny; MLCC; 1nF; 50V; X7R; ±10%; SMD; 0603" H 2900 1700 50  0001 C CNN "Opis"
+F 4 "0.07894" H 2900 1700 50  0001 C CNN "Cena"
+F 5 "https://www.tme.eu/pl/details/cl10b104kb8nnnc/kondensatory-mlcc-smd-0603/samsung/" H 2900 1700 50  0001 C CNN "Link"
+F 6 "CL10B104KB8NNNC" H 2900 1700 50  0001 C CNN "Model"
+F 7 "Kondensator: ceramiczny; MLCC; 100nF; 50V; X7R; ±10%; SMD; 0603" H 2900 1700 50  0001 C CNN "Opis"
 F 8 "SAMSUNG" H 2900 1700 50  0001 C CNN "Producent"
 F 9 "SMD" H 2900 1700 50  0001 C CNN "Typ"
+F 10 "X7R" H 2900 1700 50  0001 C CNN "Dielektryk"
+F 11 "50V" H 2900 1700 50  0001 C CNN "Napięcie"
 	1    2900 1700
 	1    0    0    -1
@@
 F 2 "Capacitor_SMD:C_0603_1608Metric" H 2938 3050 50  0001 C CNN
 F 3 "~" H 2900 3200 50  0001 C CNN
-F 4 "0.05563" H 2900 3200 50  0001 C CNN "Cena"
-F 5 "https://www.tme.eu/pl/details/cl10b102kb8nnnc/kondensatory-mlcc-smd-0603/samsung/" H 2900 3200 50  0001 C CNN "Link"
-F 6 "CL10B102KB8NNNC" H 2900 3200 50  0001 C CNN "Model"
-F 7 "Kondensator: ceramiczny; MLCC; 1nF; 50V; X7R; ±10%; SMD; 0603" H 2900 3200 50  0001 C CNN "Opis"
+F 4 "0.07894" H 2900 3200 50  0001 C CNN "Cena"
+F 5 "https://www.tme.eu/pl/details/cl10b104kb8nnnc/kondensatory-mlcc-smd-0603/samsung/" H 2900 3200 50  0001 C CNN "Link"
+F 6 "CL10B104KB8NNNC" H 2900 3200 50  0001 C CNN "Model"
+F 7 "Kondensator: ceramiczny; MLCC; 100nF; 50V; X7R; ±10%; SMD; 0603" H 2900 3200 50  0001 C CNN "Opis"
 F 8 "SAMSUNG" H 2900 3200 50  0001 C CNN "Producent"
 F 9 "SMD" H 2900 3200 50  0001 C CNN "Typ"
+F 10 "X7R" H 2900 3200 50  0001 C CNN "Dielektryk"
+F 11 "50V" H 2900 3200 50  0001 C CNN "Napięcie"
 	1    2900 3200
 	1    0    0    -1
@@
 F 2 "Capacitor_SMD:C_0603_1608Metric" H 2938 4500 50  0001 C CNN
 F 3 "~" H 2900 4650 50  0001 C CNN
-F 4 "0.05563" H 2900 4650 50  0001 C CNN "Cena"
-F 5 "https://www.tme.eu/pl/details/cl10b102kb8nnnc/kondensatory-mlcc-smd-0603/samsung/" H 2900 4650 50  0001 C CNN "Link"
-F 6 "CL10B102KB8NNNC" H 2900 4650 50  0001 C CNN "Model"
-F 7 "Kondensator: ceramiczny; MLCC; 1nF; 50V; X7R; ±10%; SMD; 0603" H 2900 4650 50  0001 C CNN "Opis"
+F 4 "0.07894" H 2900 4650 50  0001 C CNN "Cena"
+F 5 "https://www.tme.eu/pl/details/cl10b104kb8nnnc/kondensatory-mlcc-smd-0603/samsung/" H 2900 4650 50  0001 C CNN "Link"
+F 6 "CL10B104KB8NNNC" H 2900 4650 50  0001 C CNN "Model"
+F 7 "Kondensator: ceramiczny; MLCC; 100nF; 50V; X7R; ±10%; SMD; 0603" H 2900 4650 50  0001 C CNN "Opis"
 F 8 "SAMSUNG" H 2900 4650 50  0001 C CNN "Producent"
 F 9 "SMD" H 2900 4650 50  0001 C CNN "Typ"
+F 10 "X7R" H 2900 4650 50  0001 C CNN "Dielektryk"
+F 11 "50V" H 2900 4650 50  0001 C CNN "Napięcie"
 	1    2900 4650
 	1    0    0    -1
@@
 F 2 "Capacitor_SMD:C_0603_1608Metric" H 2938 6000 50  0001 C CNN
 F 3 "~" H 2900 6150 50  0001 C CNN
-F 4 "0.05563" H 2900 6150 50  0001 C CNN "Cena"
-F 5 "https://www.tme.eu/pl/details/cl10b102kb8nnnc/kondensatory-mlcc-smd-0603/samsung/" H 2900 6150 50  0001 C CNN "Link"
-F 6 "CL10B102KB8NNNC" H 2900 6150 50  0001 C CNN "Model"
-F 7 "Kondensator: ceramiczny; MLCC; 1nF; 50V; X7R; ±10%; SMD; 0603" H 2900 6150 50  0001 C CNN "Opis"
+F 4 "0.07894" H 2900 6150 50  0001 C CNN "Cena"
+F 5 "https://www.tme.eu/pl/details/cl10b104kb8nnnc/kondensatory-mlcc-smd-0603/samsung/" H 2900 6150 50  0001 C CNN "Link"
+F 6 "CL10B104KB8NNNC" H 2900 6150 50  0001 C CNN "Model"
+F 7 "Kondensator: ceramiczny; MLCC; 100nF; 50V; X7R; ±10%; SMD; 0603" H 2900 6150 50  0001 C CNN "Opis"
 F 8 "SAMSUNG" H 2900 6150 50  0001 C CNN "Producent"
 F 9 "SMD" H 2900 6150 50  0001 C CNN "Typ"
+F 10 "X7R" H 2900 6150 50  0001 C CNN "Dielektryk"
+F 11 "50V" H 2900 6150 50  0001 C CNN "Napięcie"
 	1    2900 6150
 	1    0    0    -1
@@
 F 2 "Capacitor_SMD:C_0603_1608Metric" H 9788 1500 50  0001 C CNN
 F 3 "~" H 9750 1650 50  0001 C CNN
-F 4 "0.05563" H 9750 1650 50  0001 C CNN "Cena"
-F 5 "https://www.tme.eu/pl/details/cl10b102kb8nnnc/kondensatory-mlcc-smd-0603/samsung/" H 9750 1650 50  0001 C CNN "Link"
-F 6 "CL10B102KB8NNNC" H 9750 1650 50  0001 C CNN "Model"
-F 7 "Kondensator: ceramiczny; MLCC; 1nF; 50V; X7R; ±10%; SMD; 0603" H 9750 1650 50  0001 C CNN "Opis"
+F 4 "0.07894" H 9750 1650 50  0001 C CNN "Cena"
+F 5 "https://www.tme.eu/pl/details/cl10b104kb8nnnc/kondensatory-mlcc-smd-0603/samsung/" H 9750 1650 50  0001 C CNN "Link"
+F 6 "CL10B104KB8NNNC" H 9750 1650 50  0001 C CNN "Model"
+F 7 "Kondensator: ceramiczny; MLCC; 100nF; 50V; X7R; ±10%; SMD; 0603" H 9750 1650 50  0001 C CNN "Opis"
 F 8 "SAMSUNG" H 9750 1650 50  0001 C CNN "Producent"
 F 9 "SMD" H 9750 1650 50  0001 C CNN "Typ"
+F 10 "X7R" H 9750 1650 50  0001 C CNN "Dielektryk"
+F 11 "50V" H 9750 1650 50  0001 C CNN "Napięcie"
 	1    9750 1650
 	1    0    0    -1
@@
 F 3 "~" H 8950 1850 50  0001 C CNN
 F 4 "0.04651" H 8950 1850 50  0001 C CNN "Cena"
+F 5 "https://www.tme.eu/pl/details/smd0603-100k-1%25/rezystory-smd-0603/royal-ohm/0603saf1003t5e/" H 8950 1850 50  0001 C CNN "Link"
+F 6 "0603SAF1003T5E" H 8950 1850 50  0001 C CNN "Model"
+F 7 "Rezystor: thick film; SMD; 0603; 100kΩ; 0,1W; ±1%; -55÷155°C" H 8950 1850 50  0001 C CNN "Opis"
+F 8 "ROYAL OHM" H 8950 1850 50  0001 C CNN "Producent"
+F 9 "SMD" H 8950 1850 50  0001 C CNN "Typ"
 	1    8950 1850
 	1    0    0    -1
@@
 F 4 "0.04651" H 6350 1100 50  0001 C CNN "Cena"
 F 5 "SMD" H 6350 1100 50  0001 C CNN "Typ"
+F 6 "https://www.tme.eu/pl/details/0603saj0000t5e/rezystory-smd-0603/royal-ohm/" H 6350 1100 50  0001 C CNN "Link"
+F 7 "0603SAJ0000T5E" H 6350 1100 50  0001 C CNN "Model"
+F 8 "Rezystor: thick film; SMD; 0603; 0Ω; 0,1W; ±5%; -55÷155°C; 400ppm/°C" H 6350 1100 50  0001 C CNN "Opis"
+F 9 "ROYAL OHM" H 6350 1100 50  0001 C CNN "Producent"
 	1    6350 1100
 	0    -1   -1   0
@@
 F 4 "0.04651" H 6350 1800 50  0001 C CNN "Cena"
 F 5 "SMD" H 6350 1800 50  0001 C CNN "Typ"
+F 6 "https://www.tme.eu/pl/details/0603saj0000t5e/rezystory-smd-0603/royal-ohm/" H 6350 1800 50  0001 C CNN "Link"
+F 7 "0603SAJ0000T5E" H 6350 1800 50  0001 C CNN "Model"
+F 8 "Rezystor: thick film; SMD; 0603; 0Ω; 0,1W; ±5%; -55÷155°C; 400ppm/°C" H 6350 1800 50  0001 C CNN "Opis"
+F 9 "ROYAL OHM" H 6350 1800 50  0001 C CNN "Producent"
 	1    6350 1800
 	0    -1   -1   0
@@
 F 4 "0.04651" H 6350 1900 50  0001 C CNN "Cena"
 F 5 "SMD" H 6350 1900 50  0001 C CNN "Typ"
+F 6 "https://www.tme.eu/pl/details/0603saj0000t5e/rezystory-smd-0603/royal-ohm/" H 6350 1900 50  0001 C CNN "Link"
+F 7 "0603SAJ0000T5E" H 6350 1900 50  0001 C CNN "Model"
+F 8 "Rezystor: thick film; SMD; 0603; 0Ω; 0,1W; ±5%; -55÷155°C; 400ppm/°C" H 6350 1900 50  0001 C CNN "Opis"
+F 9 "ROYAL OHM" H 6350 1900 50  0001 C CNN "Producent"
 	1    6350 1900
 	0    -1   -1   0
